File: PCB/Miirin.kicad_sch (KiCad schematic)
At the start: 27 parts, among them J1 Conn_01x04_Socket, J2 AudioJack3_Switch, Q1 Q_PMOS_GDS, SW1 SW_Push, SW2 SW_Push, SW3 SW_Push, SW4 SW_Push, SW5 SW_Push, SW6 RotaryEncoder, U1 XIAO-ESP32-S3-THT, U2 DFR0768, U3 PCF8574P

Commit message: Updated the PCB design and CAD file with the new one. Added .stl file of the case. Updated the BOM in BOM.csv and README.md
Parts:
- removed H4: MountingHole, MountingHole:MountingHole_2.2mm_M2, symbol Mechanical:MountingHole
- removed SW6: RotaryEncoder, Rotary_Encoder:RotaryEncoder_Alps_EC11E-Switch_Vertical_H20mm, symbol Device:RotaryEncoder
- added SW6: RotaryEncoder_Switch, Rotary_Encoder:RotaryEncoder_Alps_EC11E-Switch_Vertical_H20mm, symbol Device:RotaryEncoder_Switch
- SW1, SW2, SW3, SW4: footprint Button_Switch_THT:SW_PUSH_6mm -> Button_Switch_Keyboard:SW_Cherry_MX_1.00u_PCB
Connections:
- net GND: now also SW6.C, SW6.S2
- net RoEn B: now also SW6.B
- net RoEn C: now also SW6.A
- net RoEn S1: now reaches U1.9 (D8)
- net RoEn S1: now also SW6.S1
- no-connect marks 16 -> 15
Changed lines of the file:
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@@
 	)
 	(no_connect
-		(at 101.6 72.39)
-	)
-	(no_connect
 		(at 81.28 40.64)
 	)
@@
 	)
 	(label "RoEn B"
-		(at 154.94 53.34 180)
+		(at 171.45 69.85 0)
 		(effects
 			(font
 				(size 1.27 1.27)
 			)
-			(justify right bottom)
+			(justify left bottom)
 		)
 	)
@@
 		)
 	)
+	(label "RoEn S1"
+		(at 101.6 72.39 0)
+		(effects
+			(font
+				(size 1.27 1.27)
+			)
+			(justify left bottom)
+		)
+	)
 	(label "DFP Vin"
 		(at 138.43 95.25 180)
@@
 	)
 	(label "RoEn C"
-		(at 154.94 50.8 180)
+		(at 171.45 74.93 0)
 		(effects
 			(font
 				(size 1.27 1.27)
 			)
-			(justify right bottom)
+			(justify left bottom)
 		)
 	)
@@
 		)
 	)
+	(label "RoEn S1"
+		(at 156.21 74.93 180)
+		(effects
+			(font
+				(size 1.27 1.27)
+			)
+			(justify right bottom)
+		)
+	)
 	(label "SCL"
 		(at 48.26 125.73 0)
@@
 	)
 	(symbol
-		(lib_id "Mechanical:MountingHole")
-		(at 26.67 49.53 0)
-		(unit 1)
-		(body_style 1)
-		(exclude_from_sim no)
-		(in_bom no)
-		(on_board yes)
-		(in_pos_files yes)
-		(dnp no)
-		(fields_autoplaced yes)
-		(property "Reference" "H4"
-			(at 29.21 48.2599 0)
-			(show_name no)
-			(do_not_autoplace no)
-			(effects
-				(font
-					(size 1.27 1.27)
-				)
-				(justify left)
-			)
-		)
-		(property "Value" "MountingHole"
-			(at 29.21 50.7999 0)
-			(show_name no)
-			(do_not_autoplace no)
-			(effects
-				(font
-					(size 1.27 1.27)
-				)
-				(justify left)
-			)
-		)
-		(property "Footprint" "MountingHole:MountingHole_2.2mm_M2"
-			(at 26.67 49.53 0)
-			(hide yes)
-			(show_name no)
-			(do_not_autoplace no)
-			(effects
-				(font
-					(size 1.27 1.27)
-				)
-			)
-		)
-		(property "Datasheet" ""
-			(at 26.67 49.53 0)
-			(hide yes)
-			(show_name no)
-			(do_not_autoplace no)
-			(effects
-				(font
-					(size 1.27 1.27)
-				)
-			)
-		)
-		(property "Description" "Mounting Hole without connection"
-			(at 26.67 49.53 0)
-			(hide yes)
-			(show_name no)
-			(do_not_autoplace no)
-			(effects
-				(font
-					(size 1.27 1.27)
-				)
-			)
-		)
-		(instances
-			(project "Miirin"
-				(path "/ee3c5709-4871-4257-bad5-ce6d991bebad"
-					(reference "H4")
-					(unit 1)
-				)
-			)
-		)
-	)
-	(symbol
 		(lib_id "power:+3V3")
 		(at 45.72 80.01 180)
@@
 	)
 	(symbol
+		(lib_id "Device:RotaryEncoder_Switch")
+		(at 163.83 72.39 180)
+		(unit 1)
+		(body_style 1)
+		(exclude_from_sim no)
+		(in_bom yes)
+		(on_board yes)
+		(in_pos_files yes)
+		(dnp no)
+		(fields_autoplaced yes)
+		(property "Reference" "SW6"
+			(at 163.83 62.23 0)
+			(show_name no)
+			(do_not_autoplace no)
+			(effects
+				(font
+					(size 1.27 1.27)
+				)
+			)
+		)
+		(property "Value" "RotaryEncoder_Switch"
+			(at 163.83 64.77 0)
+			(show_name no)
+			(do_not_autoplace no)
+			(effects
+				(font
+					(size 1.27 1.27)
+				)
+			)
+		)
+		(property "Footprint" "Rotary_Encoder:RotaryEncoder_Alps_EC11E-Switch_Vertical_H20mm"
+			(at 167.64 76.454 0)
+			(hide yes)
+			(show_name no)
+			(do_not_autoplace no)
+			(effects
+				(font
+					(size 1.27 1.27)
+				)
+			)
+		)
+		(property "Datasheet" ""
+			(at 163.83 78.994 0)
+			(hide yes)
+			(show_name no)
+			(do_not_autoplace no)
+			(effects
+				(font
+					(size 1.27 1.27)
+				)
+			)
+		)
+		(property "Description" "Rotary encoder, dual channel, incremental quadrate outputs, with switch"
+			(at 163.83 72.39 0)
+			(hide yes)
+			(show_name no)
+			(do_not_autoplace no)
+			(effects
+				(font
+					(size 1.27 1.27)
+				)
+			)
+		)
+		(pin "A"
+		)
+		(pin "S1"
+		)
+		(pin "B"
+		)
+		(pin "C"
+		)
+		(pin "S2"
+		)
+		(instances
+			(project "Miirin"
+				(path "/ee3c5709-4871-4257-bad5-ce6d991bebad"
+					(reference "SW6")
+					(unit 1)
+				)
+			)
+		)
+	)
+	(symbol
 		(lib_id "DFR0768:DFR0768")
 		(at 165.1 96.52 0)
@@
 			)
 		)
-		(property "Footprint" "Button_Switch_THT:SW_PUSH_6mm"
+		(property "Footprint" "Button_Switch_Keyboard:SW_Cherry_MX_1.00u_PCB"
 			(at 121.92 35.56 0)
 			(hide yes)
@@
 	(symbol
 		(lib_id "power:GND")
-		(at 154.94 48.26 270)
+		(at 171.45 72.39 90)
 		(unit 1)
 		(body_style 1)
@@
 		(fields_autoplaced yes)
 		(property "Reference" "#PWR014"
-			(at 148.59 48.26 0)
+			(at 177.8 72.39 0)
 			(hide yes)
 			(show_name no)
@@
 		)
 		(property "Value" "GND"
-			(at 151.13 48.2599 90)
+			(at 175.26 72.3901 90)
 			(show_name no)
 			(do_not_autoplace no)
@@
 		)
 		(property "Footprint" ""
-			(at 154.94 48.26 0)
+			(at 171.45 72.39 0)
 			(hide yes)
 			(show_name no)
@@
 		)
 		(property "Datasheet" ""
-			(at 154.94 48.26 0)
+			(at 171.45 72.39 0)
 			(hide yes)
 			(show_name no)
@@
 		)
 		(property "Description" "Power symbol creates a global label with name \"GND\" , ground"
-			(at 154.94 48.26 0)
+			(at 171.45 72.39 0)
 			(hide yes)
 			(show_name no)
@@
 			)
 		)
-		(property "Footprint" "Button_Switch_THT:SW_PUSH_6mm"
+		(property "Footprint" "Button_Switch_Keyboard:SW_Cherry_MX_1.00u_PCB"
 			(at 121.92 46.99 0)
 			(hide yes)
@@
 			)
 		)
-		(property "Footprint" "Button_Switch_THT:SW_PUSH_6mm"
+		(property "Footprint" "Button_Switch_Keyboard:SW_Cherry_MX_1.00u_PCB"
 			(at 121.92 24.13 0)
 			(hide yes)
@@
 	)
 	(symbol
-		(lib_id "Device:RotaryEncoder")
-		(at 162.56 50.8 0)
+		(lib_id "Device:LED_RGBA")
+		(at 74.93 135.89 0)
 		(unit 1)
 		(body_style 1)
@@
 		(dnp no)
 		(fields_autoplaced yes)
-		(property "Reference" "SW6"
-			(at 168.91 49.5299 0)
+		(property "Reference" "D1"
+			(at 74.93 121.92 0)
 			(show_name no)
 			(do_not_autoplace no)
@@
 					(size 1.27 1.27)
 				)
-				(justify left)
 			)
 		)
-		(property "Value" "RotaryEncoder"
-			(at 168.91 52.0699 0)
+		(property "Value" "LED_RGBA"
+			(at 74.93 124.46 0)
 			(show_name no)
 			(do_not_autoplace no)
@@
 					(size 1.27 1.27)
 				)
-				(justify left)
 			)
 		)
-		(property "Footprint" "Rotary_Encoder:RotaryEncoder_Alps_EC11E-Switch_Vertical_H20mm"
-			(at 158.75 46.736 0)
+		(property "Footprint" "LED_THT:LED_D5.0mm-4_RGB"
+			(at 74.93 137.16 0)
 			(hide yes)
 			(show_name no)
@@
 		)
 		(property "Datasheet" ""
-			(at 162.56 44.196 0)
+			(at 74.93 137.16 0)
 			(hide yes)
 			(show_name no)
@@
 			)
 		)
-		(property "Description" "Rotary encoder, dual channel, incremental quadrate outputs"
-			(at 162.56 50.8 0)
+		(property "Description" "RGB LED, red/green/blue/anode"
+			(at 74.93 135.89 0)
 			(hide yes)
 			(show_name no)
@@
 			)
 		)
-		(pin "A"
+		(pin "2"
 		)
-		(pin "C"
+		(pin "1"
 		)
-		(pin "B"
+		(pin "4"
+		)
+		(pin "3"
 		)
 		(instances
 			(project "Miirin"
 				(path "/ee3c5709-4871-4257-bad5-ce6d991bebad"
-					(reference "SW6")
+					(reference "D1")
 					(unit 1)
 				)
@@
 	)
 	(symbol
-		(lib_id "Device:LED_RGBA")
-		(at 74.93 135.89 0)
+		(lib_id "power:GND")
+		(at 156.21 69.85 270)
 		(unit 1)
 		(body_style 1)
@@
 		(dnp no)
 		(fields_autoplaced yes)
-		(property "Reference" "D1"
-			(at 74.93 121.92 0)
+		(property "Reference" "#PWR019"
+			(at 149.86 69.85 0)
+			(hide yes)
 			(show_name no)
 			(do_not_autoplace no)
@@
 			)
 		)
-		(property "Value" "LED_RGBA"
-			(at 74.93 124.46 0)
+		(property "Value" "GND"
+			(at 152.4 69.8499 90)
 			(show_name no)
 			(do_not_autoplace no)
@@
 					(size 1.27 1.27)
 				)
+				(justify right)
 			)
 		)
-		(property "Footprint" "LED_THT:LED_D5.0mm-4_RGB"
-			(at 74.93 137.16 0)
+		(property "Footprint" ""
+			(at 156.21 69.85 0)
 			(hide yes)
 			(show_name no)
@@
 		)
 		(property "Datasheet" ""
-			(at 74.93 137.16 0)
+			(at 156.21 69.85 0)
 			(hide yes)
 			(show_name no)
@@
 			)
 		)
-		(property "Description" "RGB LED, red/green/blue/anode"
-			(at 74.93 135.89 0)
+		(property "Description" "Power symbol creates a global label with name \"GND\" , ground"
+			(at 156.21 69.85 0)
 			(hide yes)
 			(show_name no)
@@
 			)
 		)
-		(pin "2"
-		)
 		(pin "1"
 		)
-		(pin "4"
-		)
-		(pin "3"
-		)
 		(instances
 			(project "Miirin"
 				(path "/ee3c5709-4871-4257-bad5-ce6d991bebad"
-					(reference "D1")
+					(reference "#PWR019")
 					(unit 1)
 				)
@@
 			)
 		)
-		(property "Footprint" "Button_Switch_THT:SW_PUSH_6mm"
+		(property "Footprint" "Button_Switch_Keyboard:SW_Cherry_MX_1.00u_PCB"
 			(at 121.92 59.69 0)
 			(hide yes)
